Commit message: Laser scanners simulation

File: model/urdf/lms_1xx.urdf.xacro (robot description, xacro)
@@ -13,5 +13,5 @@
       <visual>
         <geometry>
-          <mesh filename="package://sick_scan/meshes/LMS1xx_small.dae" />
+          <mesh filename="package://sick_safetyscanners/model/meshes/LMS1xx_small.dae" />
         </geometry>
         <material name="blue" >
@@ -21,5 +21,5 @@
       <collision>
         <geometry>
-          <mesh filename="package://sick_scan/meshes/LMS1xx_collision.stl" />
+          <mesh filename="package://sick_safetyscanners/model/meshes/LMS1xx_collision.stl" />
         </geometry>
       </collision>
@@ -54,5 +54,5 @@
         <update_rate>${update_rate}</update_rate>
         <pose>0 0 0 0 0 0</pose>
-        <visualize>false</visualize>
+        <visualize>true</visualize>
         <ray>
           <scan>
@@ -78,4 +78,5 @@
           <topicName>${ros_topic}</topicName>
           <frameName>${link}</frameName>
+          <robotNamespace>/${name}</robotNamespace>
         </plugin>
       </sensor>
